File: Daughterboard/daughterboard.kicad_sch (KiCad schematic)
At the start: 170 parts, among them J1 USB-C 5V Sink, J2 Switched power outputs, J30 J3P Hosyond +5V_SW solder pad, J31 J3A Hosyond UART_TX solder pad, J32 J3B Hosyond UART_RX solder pad, J33 J3C Hosyond I2C_SDA solder pad, J34 J3D Hosyond I2C_SCL solder pad, J35 J3E Hosyond GPIO2 solder pad, J36 J3F Hosyond GPIO3 solder pad, J37 J3G Hosyond GPIO14 solder pad, J38 J3H Hosyond GPIO21 solder pad, J39 J3I Hosyond GND solder pad, J4 UART JST-GH 1.25mm, J40 Left gimbal B JST-GH 1.25mm, J41 Right gimbal A JST-GH 1.25mm, J42 Right gimbal B JST-GH 1.25mm, J5 I2C male header 2.54mm, J6 Deep sleep pushbutton header, J7 2S balance input JST-XH side-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, J8 Left gimbal A JST-GH 1.25mm, J91 MCP23017 GPA0 solder pad, J910 MCP23017 GPB1 solder pad, J911 MCP23017 GPB2 solder pad, J912 MCP23017 GPB3 solder pad, J913 MCP23017 GPB4 solder pad, J914 MCP23017 GPB5 solder pad, J915 MCP23017 GPB6 solder pad, J916 MCP23017 GPB7 solder pad, J92 MCP23017 GPA1 solder pad, J925 MCP23017 INTA solder pad, J926 MCP23017 INTB solder pad, J927 MCP23017 RESET solder pad, J928 MCP23017 +3V3_SW_LOGIC solder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, J929 MCP23017 GND solder pad, J93 MCP23017 GPA2 solder pad, J94 MCP23017 GPA3 solder pad, J95 MCP23017 GPA4 solder pad, J96 MCP23017 GPA5 solder pad, J97 MCP23017 GPA6 solder pad, J98 MCP23017 GPA7 solder pad, J99 MCP23017 GPB0 solder pad, Q1 CSD18502Q5B charge FET, Q2 CSD18502Q5B discharge FET, SW1 Pololu #2808 5V switch, SW2 Pololu #2808 3V3 switch, U1 BQ25887RGE 2S charger, U2 BQ28Z610DRZR-R1, U3 AP63200WU 5V Buck, U4 AP63200WU 3V3 Buck, U5 ADS1115IDGS 0x48, U6 ADS1115IDGS 0x49, U7 MCP23017-E/SO

Commit message: R17_REWORK_SPEC
Connections:
- net BAT_SYS: now also C33.1, Q2.1 (S), Q2.2 (S), Q2.3 (S), R49.2; no longer C32.1, Q1.5 (D), Q1.6 (D), Q1.7 (D), Q1.8 (D)
- net CHG_STAT: now also D2.1; no longer D2.2
- net FET_BATT_P: now also C32.1, Q1.1 (S), Q1.2 (S), Q1.3 (S), R50.2; no longer C33.1, Q2.5 (D), Q2.6 (D), Q2.7 (D), Q2.8 (D)
- net LED_CHG_A: now also D2.2; no longer D2.1
- net LED_PGOOD_A: now also D3.2; no longer D3.1
- net PG_STAT: now also D3.1; no longer D3.2
- removed net FET_SRC_COMMON: C32.2, C33.2, Q1.1 (S), Q1.2 (S), Q1.3 (S), Q2.1 (S), Q2.2 (S), Q2.3 (S), R49.2, R50.2
- new net FET_MID_COMMON: C32.2, C33.2, Q1.5 (D), Q1.6 (D), Q1.7 (D), Q1.8 (D), Q2.5 (D), Q2.6 (D), Q2.7 (D), Q2.8 (D)
Changed lines of the file:
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@@
 	(wire (pts (xy 320.04 54.61) (xy 314.96 54.61)) (stroke (width 0) (type default)))
 	(wire (pts (xy 314.96 54.61) (xy 314.96 52.07)) (stroke (width 0) (type default)))
-	(global_label "LED_CHG_A"
+	(global_label "CHG_STAT"
 		(shape bidirectional)
 		(at 314.96 52.07 0)
@@
 	(wire (pts (xy 340.36 54.61) (xy 345.44 54.61)) (stroke (width 0) (type default)))
 	(wire (pts (xy 345.44 54.61) (xy 345.44 52.07)) (stroke (width 0) (type default)))
-	(global_label "CHG_STAT"
+	(global_label "LED_CHG_A"
 		(shape bidirectional)
 		(at 345.44 52.07 0)
@@
 	(wire (pts (xy 320.04 83.82) (xy 314.96 83.82)) (stroke (width 0) (type default)))
 	(wire (pts (xy 314.96 83.82) (xy 314.96 81.28)) (stroke (width 0) (type default)))
-	(global_label "LED_PGOOD_A"
+	(global_label "PG_STAT"
 		(shape bidirectional)
 		(at 314.96 81.28 0)
@@
 	(wire (pts (xy 340.36 83.82) (xy 345.44 83.82)) (stroke (width 0) (type default)))
 	(wire (pts (xy 345.44 83.82) (xy 345.44 81.28)) (stroke (width 0) (type default)))
-	(global_label "PG_STAT"
+	(global_label "LED_PGOOD_A"
 		(shape bidirectional)
 		(at 345.44 81.28 0)
@@
 	(wire (pts (xy 288.29 199.39) (xy 283.21 199.39)) (stroke (width 0) (type default)))
 	(wire (pts (xy 283.21 199.39) (xy 283.21 196.85)) (stroke (width 0) (type default)))
-	(global_label "FET_SRC_COMMON"
+	(global_label "FET_BATT_P"
 		(shape bidirectional)
 		(at 283.21 196.85 0)
@@
 	(wire (pts (xy 288.29 194.31) (xy 283.21 194.31)) (stroke (width 0) (type default)))
 	(wire (pts (xy 283.21 194.31) (xy 283.21 191.77)) (stroke (width 0) (type default)))
-	(global_label "FET_SRC_COMMON"
+	(global_label "FET_BATT_P"
 		(shape bidirectional)
 		(at 283.21 191.77 0)
@@
 	(wire (pts (xy 288.29 189.23) (xy 283.21 189.23)) (stroke (width 0) (type default)))
 	(wire (pts (xy 283.21 189.23) (xy 283.21 186.69)) (stroke (width 0) (type default)))
-	(global_label "FET_SRC_COMMON"
+	(global_label "FET_BATT_P"
 		(shape bidirectional)
 		(at 283.21 186.69 0)
@@
 	(wire (pts (xy 323.85 199.39) (xy 328.93 199.39)) (stroke (width 0) (type default)))
 	(wire (pts (xy 328.93 199.39) (xy 328.93 196.85)) (stroke (width 0) (type default)))
-	(global_label "BAT_SYS"
+	(global_label "FET_MID_COMMON"
 		(shape bidirectional)
 		(at 328.93 196.85 0)
@@
 	(wire (pts (xy 323.85 194.31) (xy 328.93 194.31)) (stroke (width 0) (type default)))
 	(wire (pts (xy 328.93 194.31) (xy 328.93 191.77)) (stroke (width 0) (type default)))
-	(global_label "BAT_SYS"
+	(global_label "FET_MID_COMMON"
 		(shape bidirectional)
 		(at 328.93 191.77 0)
@@
 	(wire (pts (xy 323.85 189.23) (xy 328.93 189.23)) (stroke (width 0) (type default)))
 	(wire (pts (xy 328.93 189.23) (xy 328.93 186.69)) (stroke (width 0) (type default)))
-	(global_label "BAT_SYS"
+	(global_label "FET_MID_COMMON"
 		(shape bidirectional)
 		(at 328.93 186.69 0)
@@
 	(wire (pts (xy 323.85 184.15) (xy 328.93 184.15)) (stroke (width 0) (type default)))
 	(wire (pts (xy 328.93 184.15) (xy 328.93 181.61)) (stroke (width 0) (type default)))
-	(global_label "BAT_SYS"
+	(global_label "FET_MID_COMMON"
 		(shape bidirectional)
 		(at 328.93 181.61 0)
@@
 	(wire (pts (xy 339.09 199.39) (xy 334.01 199.39)) (stroke (width 0) (type default)))
 	(wire (pts (xy 334.01 199.39) (xy 334.01 196.85)) (stroke (width 0) (type default)))
-	(global_label "FET_SRC_COMMON"
+	(global_label "BAT_SYS"
 		(shape bidirectional)
 		(at 334.01 196.85 0)
@@
 	(wire (pts (xy 339.09 194.31) (xy 334.01 194.31)) (stroke (width 0) (type default)))
 	(wire (pts (xy 334.01 194.31) (xy 334.01 191.77)) (stroke (width 0) (type default)))
-	(global_label "FET_SRC_COMMON"
+	(global_label "BAT_SYS"
 		(shape bidirectional)
 		(at 334.01 191.77 0)
@@
 	(wire (pts (xy 339.09 189.23) (xy 334.01 189.23)) (stroke (width 0) (type default)))
 	(wire (pts (xy 334.01 189.23) (xy 334.01 186.69)) (stroke (width 0) (type default)))
-	(global_label "FET_SRC_COMMON"
+	(global_label "BAT_SYS"
 		(shape bidirectional)
 		(at 334.01 186.69 0)
@@
 	(wire (pts (xy 374.65 199.39) (xy 379.73 199.39)) (stroke (width 0) (type default)))
 	(wire (pts (xy 379.73 199.39) (xy 379.73 196.85)) (stroke (width 0) (type default)))
-	(global_label "FET_BATT_P"
+	(global_label "FET_MID_COMMON"
 		(shape bidirectional)
 		(at 379.73 196.85 0)
@@
 	(wire (pts (xy 374.65 194.31) (xy 379.73 194.31)) (stroke (width 0) (type default)))
 	(wire (pts (xy 379.73 194.31) (xy 379.73 191.77)) (stroke (width 0) (type default)))
-	(global_label "FET_BATT_P"
+	(global_label "FET_MID_COMMON"
 		(shape bidirectional)
 		(at 379.73 191.77 0)
@@
 	(wire (pts (xy 374.65 189.23) (xy 379.73 189.23)) (stroke (width 0) (type default)))
 	(wire (pts (xy 379.73 189.23) (xy 379.73 186.69)) (stroke (width 0) (type default)))
-	(global_label "FET_BATT_P"
+	(global_label "FET_MID_COMMON"
 		(shape bidirectional)
 		(at 379.73 186.69 0)
@@
 	(wire (pts (xy 374.65 184.15) (xy 379.73 184.15)) (stroke (width 0) (type default)))
 	(wire (pts (xy 379.73 184.15) (xy 379.73 181.61)) (stroke (width 0) (type default)))
-	(global_label "FET_BATT_P"
+	(global_label "FET_MID_COMMON"
 		(shape bidirectional)
 		(at 379.73 181.61 0)
@@
 	(wire (pts (xy 316.23 207.01) (xy 321.31 207.01)) (stroke (width 0) (type default)))
 	(wire (pts (xy 321.31 207.01) (xy 321.31 204.47)) (stroke (width 0) (type default)))
-	(global_label "FET_SRC_COMMON"
+	(global_label "FET_BATT_P"
 		(shape bidirectional)
 		(at 321.31 204.47 0)
@@
 	(wire (pts (xy 367.03 207.01) (xy 372.11 207.01)) (stroke (width 0) (type default)))
 	(wire (pts (xy 372.11 207.01) (xy 372.11 204.47)) (stroke (width 0) (type default)))
-	(global_label "FET_SRC_COMMON"
+	(global_label "BAT_SYS"
 		(shape bidirectional)
 		(at 372.11 204.47 0)
@@
 	(wire (pts (xy 295.91 222.25) (xy 290.83 222.25)) (stroke (width 0) (type default)))
 	(wire (pts (xy 290.83 222.25) (xy 290.83 219.71)) (stroke (width 0) (type default)))
-	(global_label "BAT_SYS"
+	(global_label "FET_BATT_P"
 		(shape bidirectional)
 		(at 290.83 219.71 0)
@@
 	(wire (pts (xy 316.23 222.25) (xy 321.31 222.25)) (stroke (width 0) (type default)))
 	(wire (pts (xy 321.31 222.25) (xy 321.31 219.71)) (stroke (width 0) (type default)))
-	(global_label "FET_SRC_COMMON"
+	(global_label "FET_MID_COMMON"
 		(shape bidirectional)
 		(at 321.31 219.71 0)
@@
 	(wire (pts (xy 346.71 222.25) (xy 341.63 222.25)) (stroke (width 0) (type default)))
 	(wire (pts (xy 341.63 222.25) (xy 341.63 219.71)) (stroke (width 0) (type default)))
-	(global_label "FET_BATT_P"
+	(global_label "BAT_SYS"
 		(shape bidirectional)
 		(at 341.63 219.71 0)
@@
 	(wire (pts (xy 367.03 222.25) (xy 372.11 222.25)) (stroke (width 0) (type default)))
 	(wire (pts (xy 372.11 222.25) (xy 372.11 219.71)) (stroke (width 0) (type default)))
-	(global_label "FET_SRC_COMMON"
+	(global_label "FET_MID_COMMON"
 		(shape bidirectional)
 		(at 372.11 219.71 0)
